Commit message: update

File: robot_arm.urdf (robot description, URDF)
Before this commit: robot simple_arm, 3 links, 2 joints
Links:
- added link end_effector, mass 0.1; collision sphere radius=0.02; visual sphere radius=0.02
- link base_link: mass None -> 1.0; geometry collision box size=0.2 0.2 0.05; visual box size=0.2 0.2 0.05
- link link1: mass None -> 0.5; geometry collision cylinder length=0.3 radius=0.03; visual cylinder length=0.3 radius=0.03
- link link2: mass None -> 0.3; geometry collision cylinder length=0.25 radius=0.025; visual cylinder length=0.25 radius=0.025
Joints:
- added joint end_effector_joint: type fixed, parent link2, child end_effector, origin xyz=0 0 0.25 rpy=0 0 0
- joint joint1: limit lower=-3.14 upper=3.14 effort=1 velocity=1.0 -> lower=-3.14 upper=3.14 effort=100 velocity=1.0
- joint joint2: limit lower=-3.14 upper=3.14 effort=1 velocity=1.0 -> lower=-3.14 upper=3.14 effort=100 velocity=1.0
